File: Hardware/Eagle/OpenChair.sch (EAGLE design)
At the start: 86 parts, among them IC1 7805DT, IC2 AP2112K-3.3TRG1 3.3V, Q1 12MHz 3.2x2.5, Q2 BSS84, Q3 BSS84, Q4 16MHz 3.2x2.5, SW1 RESET, U1 RJ45-8PTH, U2 NXP_LPC1768_FBD100, U3 LMC7101AIM5, U4 NRF_8001_R2Q32_T, Y1 ABS25, Y2 ABS25-32.768kHz

Commit message: Added Gerber RS274X files and updated PDF
Parts:
- C1, C2: value 18pF -> 1uF; device SparkFun-Passives:CAP0402-CAP -> SparkFun-Passives:CAP0603-CAP
- C10: value 1uF -> 12pF; device SparkFun-Passives:CAP0603-CAP -> SparkFun-Passives:CAP0402-CAP
- C11: value 0.33uF -> 12pF; device SparkFun-Passives:CAP0805 -> SparkFun-Passives:CAP0402-CAP
- C12: value 220uF 25V -> 18pF; device SparkFun-Capacitors:CAP_POLPTH1 -> SparkFun-Passives:CAP0402-CAP
- C13: value 1uF -> 18pF; device SparkFun-Passives:CAP0603-CAP -> SparkFun-Passives:CAP0402-CAP
- C14, C9: value 1uF -> 0.1uF; device SparkFun-Passives:CAP0603-CAP -> SparkFun-Passives:CAP0402-CAP
- C15, C16: value 10uF 10V -> 0.1uF; device SparkFun-Passives:CAP0603-CAP -> SparkFun-Passives:CAP0402-CAP
- C18: value 18pF -> 1.2pF
- C19: value 18pF -> 1.8pF
- C20: value 12pF -> 2.2nF
- C22: value 1.2pF -> 12pF
- C23: value 1.8pF -> 18pF
- C24: value 2.2nF -> 18pF
- C25: value 100nF -> 0.1uF
- C26: value 33nF -> 100nF
- C28: value 0.1uF -> 33nF
- C3: value 12pF -> 10uF 10V; device SparkFun-Passives:CAP0402-CAP -> SparkFun-Passives:CAP0603-CAP
- C4: value 12pF -> 0.33uF; device SparkFun-Passives:CAP0402-CAP -> SparkFun-Passives:CAP0805
- C5: value 0.1uF -> 220uF 25V; device SparkFun-Passives:CAP0402-CAP -> SparkFun-Capacitors:CAP_POLPTH1
- C6: value 0.1uF -> 10uF 10V; device SparkFun-Passives:CAP0402-CAP -> SparkFun-Passives:CAP0603-CAP
- C7, C8: value 0.1uF -> 1uF; device SparkFun-Passives:CAP0402-CAP -> SparkFun-Passives:CAP0603-CAP
- JP1: value (none) -> M10LOCK; device SparkFun-Connectors:M05LOCK -> SparkFun-Connectors:M10LOCK
- JP10: value USB_MICROB_PLUGCONN-11752 -> (none); device SparkFun-Connectors:USB_MICROB_PLUGCONN-11752 -> SparkFun-Connectors:M05LOCK
- JP11: value M10LOCK -> (none); device SparkFun-Connectors:M10LOCK -> SparkFun-Connectors:M03LOCK
- JP12: value (none) -> USB_MICROB_PLUGCONN-11752; device SparkFun-Connectors:M03LOCK -> SparkFun-Connectors:USB_MICROB_PLUGCONN-11752
- JP13: value (none) -> M02LOCK; device SparkFun-Connectors:M05LOCK -> SparkFun-Connectors:M02LOCK
- JP2: device SparkFun-Connectors:M04LOCK -> SparkFun-Connectors:M05LOCK
- JP3: device SparkFun-Connectors:M05LOCK -> SparkFun-Connectors:M04LOCK
- JP4: value (none) -> M10LOCK; device SparkFun-Connectors:M04LOCK -> SparkFun-Connectors:M10LOCK
- JP7: value M02LOCK -> M10LOCK; device SparkFun-Connectors:M02LOCK -> SparkFun-Connectors:M10LOCK
- JP8: value M10LOCK -> (none); device SparkFun-Connectors:M10LOCK -> SparkFun-Connectors:M05LOCK
- JP9: value M10LOCK -> (none); device SparkFun-Connectors:M10LOCK -> SparkFun-Connectors:M04LOCK
- Q3: value BSS84 -> 16MHz 3.2x2.5; device transistor-small-signal:BSS84 -> GHI:CRYSTAL3.2X2.5
- Q4: value 16MHz 3.2x2.5 -> BSS84; device GHI:CRYSTAL3.2X2.5 -> transistor-small-signal:BSS84
- R1: value 4.7k -> 470
- R10: value 1.5K -> 10k
- R11: value 470 -> 22k
- R14, R15: value 10k -> 4.7k
- R16: value 470 -> 10k
- R18: value 22k -> 470
- R2: value 4.7k -> 10k
- R3: value 330 -> 10k
- R4, R5: value 10k -> 33
- R6: value 33 -> 100k
- R7: value 33 -> 1k
- R8: value 1k -> 1.5K
- R9: value 100k -> 470
- U1: value RJ45-8PTH -> NXP_LPC1768_FBD100; device SparkFun-Connectors:RJ45-8PTH -> alvaroferran:NXP_LPC1768_FBD100
- U2: value NXP_LPC1768_FBD100 -> NRF_8001_R2Q32_T; device alvaroferran:NXP_LPC1768_FBD100 -> alvaroferran:NRF_8001_R2Q32_T
- U4: value NRF_8001_R2Q32_T -> RJ45-8PTH; device alvaroferran:NRF_8001_R2Q32_T -> SparkFun-Connectors:RJ45-8PTH
Connections:
- net !RST: now also R2.1, U1.!RESET; no longer R12.1, U2.!RESET
- net 3.3V: now also C14.1, C15.1, C25.1, C8.2, C9.1, JP1.1, JP1.10, JP1.2, JP1.3, JP1.4, JP1.6, JP1.7, JP1.8, JP1.9, JP10.5, JP2.5, JP3.4, JP9.4, R10.2, R14.1, R15.1, R2.2, R3.2, U1.VDD(3V3)@1, U1.VDD(3V3)@2, U1.VDD(3V3)@3, U1.VDD(3V3)@4, U1.VDD(REG)(3V3)@1, U1.VDD(REG)(3V3)@2, U2.AVDD, U2.VDD; no longer C17.2, C28.1, C5.1, C7.1, C8.1, JP13.5, JP2.4, JP3.5, JP4.4, JP8.1, JP8.10, JP8.2, JP8.3, JP8.4, JP8.6, JP8.7, JP8.8, JP8.9, R1.1, R12.2, R15.2, R2.1, R4.2, U2.VDD(3V3)@1, U2.VDD(3V3)@2, U2.VDD(3V3)@3, U2.VDD(3V3)@4, U2.VDD(REG)(3V3)@1, U2.VDD(REG)(3V3)@2, U4.AVDD, U4.VDD
- net 5V: now also C1.2, C3.1, C7.2, Q4.S; no longer C13.2, C14.2, C15.1, Q3.S
- net BTNA: now also JP13.2, U4.6; no longer JP14.2, U1.6
- net BTNB: now also JP13.1, U4.7; no longer JP14.1, U1.7
- net D+: now also JP12.D+, R5.2; no longer JP10.D+, R6.2
- net D-: now also JP12.D-, R4.2; no longer JP10.D-, R7.2
- net GND: now also C1.1, C10.2, C12.2, C13.2, C14.2, C2.1, C23.2, C25.2, C28.1, C5.-, C7.1, C8.1, C9.2, JP10.4, JP11.1, JP12.GND, JP12.SHIELD, JP4.10, JP4.2, JP4.3, JP4.4, JP4.5, JP4.6, JP4.7, JP4.8, JP4.9, JP8.1, R1.1, R11.1, R12.1, R6.2, U1.VREFN, U1.VSS1, U1.VSS2, U1.VSS3, U1.VSS4, U1.VSS5, U1.VSS6, U1.VSSA, U2.EXP, U2.VSS, U4.2, U4.4; no longer C1.2, C10.1, C12.-, C13.1, C14.1, C19.2, C2.2, C25.1, C28.2, C5.2, C7.2, C8.2, C9.1, JP1.1, JP10.GND, JP10.SHIELD, JP12.1, JP13.4, JP9.10, JP9.2, JP9.3, JP9.4, JP9.5, JP9.6, JP9.7, JP9.8, JP9.9, R14.1, R16.1, R18.1, R9.2, U1.2, U1.4, U2.VREFN, U2.VSS1, U2.VSS2, U2.VSS3, U2.VSS4, U2.VSS5, U2.VSS6, U2.VSSA, U4.EXP, U4.VSS
- net ISP: now also R3.1, U1.P2[10]/EINT0/NMI; no longer R15.1, U2.P2[10]/EINT0/NMI
- net N$1: now also JP14.2, R18.2; no longer JP7.2, R3.2
- net N$11: now also JP11.3, R17.1; no longer JP12.3, R4.1
- net N$12: now also R6.1, R7.1, U1.P1[30]/VBUS/AD0[4]; no longer R8.1, R9.1, U2.P1[30]/VBUS/AD0[4]
- net N$13: now also R5.1, R8.2, U1.P0[29]/USB_D+; no longer R10.2, R6.1, U2.P0[29]/USB_D+
- net N$14: now also R9.1, U1.P1[18]/USB_UP_LED/PWM1[1]/CAP1[0]; no longer R11.1, U2.P1[18]/USB_UP_LED/PWM1[1]/CAP1[0]
- net N$15: now also LED2.C, R9.2; no longer LED1.C, R11.2
- net N$16: now also R4.1, U1.P0[30]/USB_D-; no longer R7.1, U2.P0[30]/USB_D-
- net N$17: now also R8.1; no longer R10.1
- net N$18: now also Q4.G; no longer Q3.G
- net N$2: now also SJ3.1, U4.1; no longer SJ1.1, U1.1
- net N$20: now also R12.2; no longer R14.2
- net N$21: now also R11.2, U2.IREF; no longer R18.2, U4.IREF
- net N$22: now also C26.2, U2.DEC1; no longer C25.2, U4.DEC1
- net N$23: now also C28.2, U2.DEC2; no longer C26.2, U4.DEC2
- net N$24: now also R10.1, U2.!RESET; no longer R17.1, U4.!RESET
- net N$25: now also U2.ANT2; no longer U4.ANT2
- net N$26: now also U2.ANT1; no longer U4.ANT1
- net N$29: now also C19.1; no longer C23.1
- net N$3: now also U4.3; no longer U1.3
- net N$30: now also C18.1, C19.2; no longer C22.1, C23.2
- net N$4: now also SJ1.1, U4.5; no longer SJ3.1, U1.5
- net N$5: now also JP12.VCC; no longer JP10.VCC
- net N$6: now also JP11.2, R16.1; no longer JP12.2, R5.1
- net N$7: now also LED1.C, R1.2; no longer LED2.C, R16.2
- net P0: now also JP7.1, U1.P0[25]/AD0[2]/I2SRX_SDA/TXD3; no longer JP11.1, U2.P0[25]/AD0[2]/I2SRX_SDA/TXD3
- net P1: now also JP7.2, U1.P0[26]/AD0[3]/AOUT/RXD3; no longer JP11.2, U2.P0[26]/AD0[3]/AOUT/RXD3
- net P2: now also JP7.3, U1.P1[31]/SCK1/AD0[5]; no longer JP11.3, U2.P1[31]/SCK1/AD0[5]
- net P3: now also JP7.4, U1.P0[3]/RXD0/AD0[6]; no longer JP11.4, U2.P0[3]/RXD0/AD0[6]
- net P4: now also JP7.5, U1.P0[2]/TXD0/AD0[7]; no longer JP11.5, U2.P0[2]/TXD0/AD0[7]
- net P5: now also JP7.6, U1.P2[0]/PWM1[1]/TXD1; no longer JP11.6, U2.P2[0]/PWM1[1]/TXD1
- net P6: now also JP7.7, U1.P2[1]/PWM1[2]/RXD1; no longer JP11.7, U2.P2[1]/PWM1[2]/RXD1
- net P7: now also JP7.8, U1.P2[2]/PWM1[3]/CTS1/TRACEDATA[3]; no longer JP11.8, U2.P2[2]/PWM1[3]/CTS1/TRACEDATA[3]
- net P8: now also JP7.9, U1.P2[3]/PWM1[4]/DCD1/TRACEDATA[2]; no longer JP11.9, U2.P2[3]/PWM1[4]/DCD1/TRACEDATA[2]
- net P9: now also JP7.10, U1.P2[4]/PWM1[5]/DSR1/TRACEDATA[1]; no longer JP11.10, U2.P2[4]/PWM1[5]/DSR1/TRACEDATA[1]
- net PACT: now also U1.P2[13]/EINT3/I2STX_SDA, U2.ACTIVE; no longer U2.P2[13]/EINT3/I2STX_SDA, U4.ACTIVE
- net PJB: now also JP10.1, U1.P1[0]/ENET_TXD0; no longer JP13.1, U2.P1[0]/ENET_TXD0
- net PJX: now also JP10.3, U1.P0[24]/AD0[1]/I2SRX_WS/CAP3[1]; no longer JP13.3, U2.P0[24]/AD0[1]/I2SRX_WS/CAP3[1]
- net PJY: now also JP10.2, U1.P0[23]/AD0[0]/I2SRX_CLK/CAP3[0]; no longer JP13.2, U2.P0[23]/AD0[0]/I2SRX_CLK/CAP3[0]
- net PLG: now also R18.1, U1.P0[8]/I2STX_WS/MISO1/MAT2[2]; no longer R3.1, U2.P0[8]/I2STX_WS/MISO1/MAT2[2]
- net PLR: now also JP14.1, U1.P0[9]/I2STX_SDA/MOSI1/MAT2[3]; no longer JP7.1, U2.P0[9]/I2STX_SDA/MOSI1/MAT2[3]
- net PMISO: now also JP2.3, JP8.3, U1.P0[17]/CTS1/MISO0/MISO, U2.MISO; no longer JP1.3, JP3.3, U2.P0[17]/CTS1/MISO0/MISO, U4.MISO
- net PMOSI: now also JP2.4, JP8.4, U1.P0[18]/DCD1/MOSI0/MOSI, U2.MOSI; no longer JP1.4, JP3.4, U2.P0[18]/DCD1/MOSI0/MOSI, U4.MOSI
- net PRDY: now also U1.P2[11]/EINT1/I2STX_CLK, U2.!RDYN; no longer U2.P2[11]/EINT1/I2STX_CLK, U4.!RDYN
- net PREQ: now also U1.P2[12]/EINT2/I2STX_WS, U2.!REQN; no longer U2.P2[12]/EINT2/I2STX_WS, U4.!REQN
- net PSCK: now also JP2.2, JP8.2, U1.P0[15]/TXD1/SCK0/SCK, U2.SCK; no longer JP1.2, JP3.2, U2.P0[15]/TXD1/SCK0/SCK, U4.SCK
- net PSCL: now also JP3.2, JP9.2, R15.2, U1.P0[28]/SCL0/USB_SCL; no longer JP2.2, JP4.2, R2.2, U2.P0[28]/SCL0/USB_SCL
- net PSDA: now also JP3.3, JP9.3, R14.2, U1.P0[27]/SDA0/USB_SDA; no longer JP2.3, JP4.3, R1.2, U2.P0[27]/SDA0/USB_SDA
- net PSW: now also R16.2, U1.P0[7]/I2STX_CLK/SCK1/MAT2[1]; no longer R5.2, U2.P0[7]/I2STX_CLK/SCK1/MAT2[1]
- net RX2: now also SJ3.2, U1.P0[11]/RXD2/SCL2/MAT3[1]; no longer SJ1.2, U2.P0[11]/RXD2/SCL2/MAT3[1]
- net RX3: now also U1.P0[1]/TD1/RXD3/SCL1; no longer U2.P0[1]/TD1/RXD3/SCL1
- net RXT1: now also C11.1, U1.RTCX1; no longer C3.1, U2.RTCX1
- net RXT2: now also C10.1, U1.RTCX2; no longer C4.1, U2.RTCX2
- net TX2: now also U1.P0[10]/TXD2/SDA2/MAT3[0]; no longer U2.P0[10]/TXD2/SDA2/MAT3[0]
- net TX3: now also SJ1.2, U1.P0[0]/RD1/TXD3/SDA1; no longer SJ3.2, U2.P0[0]/RD1/TXD3/SDA1
- net USBC: now also U1.P2[9]/USB_CONNECT/RXD2/ENET_MDIO; no longer U2.P2[9]/USB_CONNECT/RXD2/ENET_MDIO
- net VBAT: now also U1.VBAT; no longer U2.VBAT
- net VCC: now also Q4.D, R7.2; no longer Q3.D, R8.2
- net VDDA: now also C17.2, U1.VDDA, U1.VREFP; no longer C9.2, U2.VDDA, U2.VREFP
- net VDD_PA: now also C20.1, U2.VDD_PA; no longer C24.1, U4.VDD_PA
- net VIN: now also C2.2, C4.1, C5.+, U4.8; no longer C10.2, C11.1, C12.+, U1.8
- net XC1: now also C24.1, Q3.P$2, U2.XC1; no longer C18.1, Q4.P$2, U4.XC1
- net XC2: now also C23.1, Q3.P$1, U2.XC2; no longer C19.1, Q4.P$1, U4.XC2
- net XL1: now also C22.1, U2.XL1; no longer C20.1, U4.XL1
- net XL2: now also U2.XL2; no longer U4.XL2
- net XT1: now also C13.1, U1.XTAL1; no longer C1.1, U2.XTAL1
- net XT2: now also C12.1, U1.XTAL2; no longer C2.1, U2.XTAL2
Other:
- moved on the sheet: C1, C10, C11, C13, C14, C15, C16, C17, C18, C19, C2, C20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
